Commit message: merged agv_control with new world

File: agv_low/robots/agv_urdf_youbot_collsionwheel.xacro (robot description, xacro)
@@ -7,5 +7,5 @@
 	<!-- Import summit XL base elements -->
 	<xacro:include filename="$(find agv_low)/urdf/bases/agv_low_base_urdf.xacro" />
-	<xacro:include filename="$(find agv_low)/urdf/bases/agv_low_base_gazebo_urdf.xacro" />
+<!--	<xacro:include filename="$(find agv_low)/urdf/bases/agv_low_base_gazebo_urdf.xacro" /> -->
 	<!-- Import summit XL wheels collision -->
 	<xacro:include filename="$(find agv_low)/urdf/wheels/agv_low_wheel_urdf_youbot_collision.xacro" />
@@ -30,8 +30,8 @@
   		<xacro:mecanum_wheel_youbot_collision prefix="${prefix}back_left" angle="-1" parent="${prefix}base_link" />
   		<xacro:mecanum_wheel_youbot_collision prefix="${prefix}back_right" angle="1" parent="${prefix}base_link" />
-		<xacro:mecanum_wheel_visual prefix="${prefix}front_left" angle="-1" wheel_pos="0" parent="${prefix}base_link" />
-  		<xacro:mecanum_wheel_visual prefix="${prefix}front_right" angle="1" wheel_pos="1" parent="${prefix}base_link" />
-  		<xacro:mecanum_wheel_visual prefix="${prefix}back_left" angle="-1" wheel_pos="1" parent="${prefix}base_link" />
-  		<xacro:mecanum_wheel_visual prefix="${prefix}back_right" angle="1" wheel_pos="0" parent="${prefix}base_link" />
+		<xacro:mecanum_wheel_visual prefix="${prefix}front_left" angle="-1" wheel_pos="1" parent="${prefix}base_link" />
+  		<xacro:mecanum_wheel_visual prefix="${prefix}front_right" angle="1" wheel_pos="0" parent="${prefix}base_link" />
+  		<xacro:mecanum_wheel_visual prefix="${prefix}back_left" angle="-1" wheel_pos="0" parent="${prefix}base_link" />
+  		<xacro:mecanum_wheel_visual prefix="${prefix}back_right" angle="1" wheel_pos="1" parent="${prefix}base_link" />
 		<!-- Gazebo ros control pluggins -->
   		<!-- IMU -->
@@ -55,6 +55,6 @@
 		</xacro:sensor_asus_xtion_pro_stand>
    	</xacro:macro>
-   <!-- Gazebo ros control plugins -->
-<!--    <xacro:ros_control />  -->
+   <!-- Gazebo ros control pluggins -->
+   <!-- <xacro:ros_control /> -->
    <!-- <xacro:ros_force_based_move prefix="$(arg prefix)"/> -->
 <!--   <xacro:planar_move prefix="$(arg prefix)"/> -->
@@ -62,16 +62,3 @@
    <xacro:agv prefix="$(arg prefix)"/>
    <!--<xacro:xtion_stand parent="agv_base_link" tilting_angle="0" /> -->
-   <!-- Gazebo ground truth odom plugin -->
-	<gazebo>
-	  <plugin name="p3d_base_controller" filename="libgazebo_ros_p3d.so">
-	    <alwaysOn>true</alwaysOn>
-	    <updateRate>25.0</updateRate>   <!-- 50 Hz -->
-	    <bodyName>agv_base_link</bodyName>
-	    <topicName>/agv_mecanum/ground_truth/state</topicName>
-	    <gaussianNoise>0.01</gaussianNoise>
-	    <frameName>map</frameName>
-	    <xyzOffset>0 0 0</xyzOffset>
-	    <rpyOffset>0 0 0</rpyOffset>
-	  </plugin>
-	</gazebo>
 </robot>

File: agv_low/urdf/bases/agv_low_base_gazebo_urdf.xacro (robot description, xacro)
@@ -4,12 +4,13 @@
   <xacro:macro name="ros_control">
     <gazebo>
-      <plugin name="ros_control" filename="libgazebo_ros_control.so">
+      <plugin name="gazebo_ros_control" filename="libgazebo_ros_control.so">
         <!--<robotNamespace>/agv_low</robotNamespace>-->
 <!--	<robotParam>robot_description</robotParam>
         <controlPeriod>0.001</controlPeriod> -->
 	<robotSimType>gazebo_ros_control/DefaultRobotHWSim</robotSimType>
+        <legacyModeNS>true</legacyModeNS>
       </plugin>
     </gazebo>
-	</xacro:macro>
+  </xacro:macro>
 <!--
   <xacro:macro name="omni_steering" params="prefix">
@@ -39,5 +40,5 @@
 			 <odometryRate>50.0</odometryRate>
 			 <publishOdometryTf>true</publishOdometryTf>
-		 </plugin>
+		 </plugin>    <legacyModeNS>true</legacyModeNS>
 	  </gazebo>
   </xacro:macro>

File: agv_low/urdf/bases/agv_low_base_urdf.xacro (robot description, xacro)
@@ -12,5 +12,5 @@
 	</link>
 	<joint name="${prefix}base_footprint_joint" type="fixed">
-		<origin xyz="0 0 0.338" rpy="0 0 0" /> <!-- "0.48 -0.0245 0" -->
+		<origin xyz="0 0 0.338" rpy="0 0 3.14" /> <!-- "0.48 -0.0245 0" -->
 		<parent link="${prefix}base_footprint"/>
 		<child link="${prefix}base_link" />

File: agv_low/urdf/ros_controller.urdf.xacro (robot description, xacro)
@@ -3,5 +3,6 @@
   <gazebo>
     <plugin name="gazebo_ros_controller" filename="libgazebo_ros_control.so" />
-    	<robotNamespace>agv_steeredwheel</robotNamespace>
+        <legacyModeNS>true</legacyModeNS>
+    <!--	<robotNamespace>agv_steeredwheel</robotNamespace> -->
   </gazebo>
 </robot>

File: agv_low/urdf/sensors/sick_s300.urdf.xacro (robot description, xacro)
@@ -13,5 +13,5 @@
 				<!--<box size="0.106 0.094 0.152"/>-->
 				<!--<cylinder radius="0.058" length="0.152"/>-->
-	     		<mesh filename="package://robotnik_sensors/meshes/sick_s300.dae"/>
+	     		<mesh filename="package://agv_low/meshes/sensors/sick.obj"/>
 			</geometry>
 		</collision>
@@ -19,5 +19,5 @@
 			<origin xyz="0 0 0" rpy="0 0 0"/>
 			<geometry>
-	     		<mesh filename="package://robotnik_sensors/meshes/sick_s300.dae"/>
+	     		<mesh filename="package://agv_low/meshes/sensors/sick.obj"/>
 			</geometry>
 		</visual>
